Commit message: fix: align wheelchair kinematics and runtime lifecycle handling

File: ros2/src/wheelchair_description/urdf/joints.xacro (robot description, xacro)
@@ -5,5 +5,5 @@
     <child link="left_wheel"/>
     <origin xyz="0.02 0.31 -0.04" rpy="1.5708 0 0"/>
-    <axis xyz="0 1 0"/>
+    <axis xyz="0 0 -1"/>
   </joint>
   <joint name="right_wheel_joint" type="continuous">
@@ -11,5 +11,5 @@
     <child link="right_wheel"/>
     <origin xyz="0.02 -0.31 -0.04" rpy="1.5708 0 0"/>
-    <axis xyz="0 1 0"/>
+    <axis xyz="0 0 -1"/>
   </joint>
   <joint name="caster_left_joint" type="fixed">
